File: cockatiel/hardware/version/cockatiel.kicad_pcb (KiCad board)
At the start: 2 copper layers, 113.8 x 72.9 mm, 17 parts, among them J1 USB_C_Receptacle_USB2.0

Commit message: commit bc im formatting my pc lol
Other:
- copper layers 2 -> 4
- rule pad_to_mask_clearance: 0 -> 0.05
