File: cockatiel/hardware/version/cockatiel.kicad_sch (KiCad schematic)
At the start: 55 parts, among them J1 USB_C_Receptacle_USB2.0, J2 Sea-Picro, Q1 2N7002VC-7, Q2 2N7002VC-7, SW1 SWITCH, U1 XC6210B332MR-G, U2 GD25Q64CWIGR, U3 RP2040, Y1 12MHz

Commit message: commit bc im formatting my pc lol
Parts:
- removed C1, C2, C3, C6: 4u7, Capacitor_SMD:C_0402_1005Metric, symbol Device:C
- removed C10, C13: 1u, Capacitor_SMD:C_0402_1005Metric, symbol Device:C
- removed C11, C12, C14, C15, C16, C17, C18, C19, C5, C9: 100n, Capacitor_SMD:C_0402_1005Metric, symbol Device:C
- removed C4: 10u, Capacitor_SMD:C_0402_1005Metric, symbol Device:C
- removed C7, C8: 15p, Capacitor_SMD:C_0402_1005Metric, symbol Device:C
- removed D1: B5817WS, josh-passives-smt:D_SOD-323, symbol Device:D_Schottky
- removed D2: LED, LED_SMD:LED_0603_1608Metric, symbol Device:LED
- removed D3: WS2812C-2020, josh-led:WS2812C-2020, symbol josh-led:WS2812C-2020
- removed F1: 500mA, josh-passives-smt:Fuse_0603_1608Metric, symbol Device:Polyfuse_Small
- removed J1: USB_C_Receptacle_USB2.0, josh-connectors:USB-C_MID_MOUNT_918-418K2024S40000, symbol josh-connector:USB_C_Receptacle_USB2.0_NO_SBU
- removed J2: Sea-Picro, josh-module:Sea-Picro_RST_Pins, symbol josh-module:Sea-Picro
- removed LOGO1: Sea-Picro, josh-logos:sea-picro-silk, symbol Graphic:SYM_LASER_Small
- removed LOGO2: Logo_Open_Hardware_Small, josh-logos:OSHW_Logo_3.6x3.6_F.Mask, symbol Graphic:Logo_Open_Hardware_Small
- removed Q1, Q2: 2N7002VC-7, josh-soic-sot-etc:SOT-563, symbol Transistor_FET:FDG6335N
- removed R1, R10, R11, R16, R2, R3, R4, R5: 5K1, Resistor_SMD:R_0402_1005Metric, symbol Device:R
- removed R12, R13: 27R, Resistor_SMD:R_0402_1005Metric, symbol Device:R
- removed R14, R9: 1K, Resistor_SMD:R_0402_1005Metric, symbol Device:R
- removed R15, R17: 2K2, Resistor_SMD:R_0402_1005Metric, symbol Device:R
- removed R6, R7, R8: 51K, Resistor_SMD:R_0402_1005Metric, symbol Device:R
- removed SW1: SWITCH, josh-buttons-switches:SW_Push_KMR2, symbol Switch:SW_Push
- removed TP1: nRST, josh-test-point:TestPoint_SMDPad_D1.0mm_NO_SILK, symbol Connector:TestPoint
- removed TP2: BOOT, josh-test-point:TestPoint_SMDPad_D1.0mm_NO_SILK, symbol Connector:TestPoint
- removed TP3: CLK, josh-test-point:TestPoint_THTPad_D1.0mm_Drill0.5mm_NO_SILK, symbol Connector:TestPoint
- removed TP4: IO, josh-test-point:TestPoint_THTPad_D1.0mm_Drill0.5mm_NO_SILK, symbol Connector:TestPoint
- removed U1: XC6210B332MR-G, josh-soic-sot-etc:SOT-23-5, symbol Regulator_Linear:AP2112K-3.3
- removed U2: GD25Q64CWIGR, josh-dfn-qfn:WSON-8-1EP_6x5mm_P1.27mm_EP3.4x4mm, symbol josh-memory:W25Q128JVSIQ
- removed U3: RP2040, josh-dfn-qfn:RP2040-QFN-56, symbol josh-ic:RP2040
- removed Y1: 12MHz, josh-oscillators:Crystal_SMD_2520-4Pin_2.5x2.0mm, symbol Device:Crystal_GND24_Small
- added C? (x2): 15pF, MirFol_db_local.DbLib:CAP_0402_R, symbol Femto_module-altium-import:1_CAP
- added C? (x9): 100nF, MirFol_db_local.DbLib:CAP_0402_R, symbol Femto_module-altium-import:1_CAP
- added C? (x4): 2.2uF, MirFol_db_local.DbLib:CAP_0402_R, symbol Femto_module-altium-import:1_CAP
- added LED?: Red, Pineberry_Lib.PcbLib:LED_0402_R, symbol Femto_module-altium-import:1_DIO_LED_RED
- added MOD?: LGA40 Module (Reversed!), Pineberry_Lib.PcbLib:PCB_LGA40_120X120_P100_REV, symbol Femto_module-altium-import:0_PCB_LGA40_P100
- added R?: 2k, MirFol_db_local.DbLib:RES_0402_R, symbol Femto_module-altium-import:1_RES
- added R?: 100R, MirFol_db_local.DbLib:RES_0402_R, symbol Femto_module-altium-import:2_RES
- added R?: 1k, MirFol_db_local.DbLib:RES_0402_R, symbol Femto_module-altium-import:3_RES
- added R? (x2): 10k, MirFol_db_local.DbLib:RES_0402_R, symbol Femto_module-altium-import:1_RES
- added R?: 1k, MirFol_db_local.DbLib:RES_0402_R, symbol Femto_module-altium-import:1_RES
- added U?: W25Q16JV, USON8_footprint.PcbLib:ICC_USON8_200X300X55P50_EP, symbol Femto_module-altium-import:0_ICC_WBD_W25Q64_SOIC_WSON_USON
- added U?: RP2040, MirFol_db_local.DbLib:ICC_QFN56_700X700X90_P40_EP_RP2040, symbol Femto_module-altium-import:0_ICC_RPI_RP2040_QFN56
- added X?: 12.000MHz, Pineberry_Lib.PcbLib:OSC_2520_4P_250X200H50_R, symbol Femto_module-altium-import:0_OSC_XTL_P4
Connections:
- net GND: now also C?.1, C?.1, C?.1, C?.1, C?.1, C?.1, C?.1, C?.1, C?.1, C?.1, C?.1, C?.1, C?.1, C?.1, C?.1, MOD?.1 (1_(CR)), MOD?.12 (12_(CR)), MOD?.23 (23_(CR)), MOD?.34 (34_(CR)), MOD?.6, MOD?.9, R?.1, U?.19 (TESTEN), U?.4 (GND), U?.EP, U?.EP (GND(EP)), X?.2, X?.4
- new net: LED?.1, R?.2
- new net: C?.2, R?.2, X?.1
- new net BOOTSEL: MOD?.3, R?.1
- new net GPIO0: MOD?.44, U?.2 (GPIO0)
- new net GPIO1: MOD?.2, U?.3 (GPIO1)
- new net GPIO10: MOD?.35, U?.13 (GPIO10)
- new net GPIO11: MOD?.33, U?.14 (GPIO11)
- new net GPIO12: MOD?.32, U?.15 (GPIO12)
- new net GPIO13: MOD?.31, U?.16 (GPIO13)
- new net GPIO14: MOD?.30, U?.17 (GPIO14)
- new net GPIO15: MOD?.29, U?.18 (GPIO15)
- new net GPIO16: MOD?.25, U?.27 (GPIO16)
- new net GPIO17: MOD?.24, U?.28 (GPIO17)
- new net GPIO18: MOD?.22, U?.29 (GPIO18)
- new net GPIO19: MOD?.21, U?.30 (GPIO19)
- new net GPIO2: MOD?.43, U?.4 (GPIO2)
- new net GPIO20: MOD?.20, U?.31 (GPIO20)
- new net GPIO21: MOD?.19, U?.32 (GPIO21)
- new net GPIO22: MOD?.18, U?.34 (GPIO22)
- new net GPIO23: MOD?.17, U?.35 (GPIO23)
- new net GPIO24: MOD?.16, U?.36 (GPIO24)
- new net GPIO25: MOD?.15, U?.37 (GPIO25)
- new net GPIO26_ADC0: MOD?.14, U?.38 (GPIO26/ADC0)
- new net GPIO27_ADC1: MOD?.13, U?.39 (GPIO27/ADC1)
- new net GPIO28_ADC2: MOD?.10, U?.40 (GPIO28/ADC2)
- new net GPIO29_ADC3: MOD?.11, U?.41 (GPIO29/ADC3)
- new net GPIO3: MOD?.42, U?.5 (GPIO3)
- new net GPIO4: MOD?.41, U?.6 (GPIO4)
- new net GPIO5: MOD?.40, U?.7 (GPIO5)
- new net GPIO6: MOD?.39, U?.8 (GPIO6)
- new net GPIO7: MOD?.38, U?.9 (GPIO7)
- new net GPIO8: MOD?.37, U?.11 (GPIO8)
- new net GPIO9: MOD?.36, U?.12 (GPIO9)
- new net MCU_RUN: MOD?.26, R?.1, U?.26 (RUN)
- new net MCU_SWCLK: MOD?.28, U?.24 (SWCLK)
- new net MCU_SWDIO: MOD?.27, U?.25 (SWDIO)
- new net MCU_XIN: C?.2, U?.20 (XIN), X?.3
- new net MCU_XOUT: R?.1, U?.21 (XOUT)
- new net PP1100: C?.2, C?.2, C?.2, U?.23 (DVDD), U?.45 (VREG_VOUT), U?.50 (DVDD)
- new net PP3300: C?.2, C?.2, C?.2, C?.2, C?.2, C?.2, C?.2, C?.2, C?.2, LED?.2, MOD?.4, MOD?.5, R?.2, R?.2, R?.2, U?.1 (IOVDD), U?.10 (IOVDD), U?.22 (IOVDD), U?.33 (IOVDD), U?.42 (IOVDD), U?.44 (VREG_VIN), U?.48 (USB_VDD), U?.49 (IOVDD), U?.8 (VCC)
- new net PP3300_AVDD: C?.2, R?.1, U?.43 (ADC_AVDD)
- new net QSPI_SCLK: U?.52 (QSPI_SCLK), U?.6 (CLK)
- new net QSPI_SD0: U?.5 (DI_(IO0)), U?.53 (QSPI_SD0)
- new net QSPI_SD1: U?.2 (DO_(IO1)), U?.55 (QSPI_SD1)
- new net QSPI_SD2: U?.3 (~{WP}_(IO2)), U?.54 (QSPI_SD2)
- new net QSPI_SD3: U?.51 (QSPI_SD3), U?.7 (~{HOLD}_(IO3))
- new net QSPI_SS: R?.1, R?.2, U?.1 (~{CS), U?.56 (QSPI_SS_N)
- new net USB_N: MOD?.8, U?.46 (USB_DM)
- new net USB_P: MOD?.7, U?.47 (USB_DP)
- no-connect marks 17 -> 0
Other:
- note added: "4-64Mbit Flash, Quad SPI, 100-133MHz, XIP (eXecute In Place), USON 2x3mm, 3.3V: Winbond: W25Q16JVUXIQ (2MB, 133 MHz) GigaDevice: GD25Q40CEIGR (512kB, 120MHz) GigaDevice: GD25Q80CEIGR (1MB, 120 MHz) GigaDevice: GD25Q80EEIGR (1MB, 133MHz) ISSI: IS25LP080D-JULE (1MB, 133 MHz)"
- note added: "ADC_AVDD"
- note added: "BOM:"
- note added: "BOOT"
- note added: "Crystal 12MHz, 2520 SMD package: JYJE: 2TJ412000NYGBC JGHC: S22120001210120 Yangxing Tech: X252012MMB4SI-24 Seiko Epson: Q24FA20H0068700 ECS: ECS-120-12-36-AGN-TR3"
- note added: "DECOUPLING CAPACITORS"
- note added: "DVDD"
- note added: "IOVDD & USB_VDD"
- note added: "OSC"
- note added: "QSPI FLASH"
- note added: "RESET"
- note added: "RP2040 MCU"
- note added: "To optional switch"
- note added: "VREG_IN"
- note added: "VREG_OUT"
- note removed: "IO"
- note removed: "LEDs"
- note removed: "Place caps close to VREG_VIN and VREG_VOUT"
- note removed: "Power"
- note removed: "Q1A - inverter, as button can only pull to ground due to being backwards compatiable"
- note removed: "Q1B - using body diode due to lack of space. Can sub with normal diode"
- note removed: "Q2A - pulls nRST to GND"
- note removed: "Q2B - pulls nCS to GND"
- note removed: "RC delay"
- note removed: "RP2040"
- note removed: "Reset / Boot Circuit"
- note removed: "Tap for < 500ms to reset Hold for > 500ms to enter UF2 bootloader"
- note removed: "USB"
